Commit message: fully functioned robotic hand, need to fix how to send to the arduino.  split them using semicolon

File: arduinobot_ws/src/arduinobot_description/urdf/arduinobot.urdf.xacro (robot description, xacro)
@@ -1,4 +1,5 @@
 <?xml version="1.0"?>
 <robot xmlns:xacro="http://www.ros.org/wiki/xacro" name="arduinobot">
+    <xacro:arg name="is_sim" default="true"/>
     <xacro:include filename="$(find arduinobot_description)/urdf/arduinobot_gazebo.xacro" />
     <xacro:include filename="$(find arduinobot_description)/urdf/arduinobot_ros2_control.xacro" />

File: arduinobot_ws/src/arduinobot_description/urdf/arduinobot_ros2_control.xacro (robot description, xacro)
@@ -3,7 +3,23 @@
     <xacro:property name="PI" value="3.14159"/>
     <ros2_control name="RobotSystem" type="system">
-        <hardware>
-            <plugin>gazebo_ros2_control/GazeboSystem</plugin>
-        </hardware>
+        <xacro:if value="$(arg is_sim)">
+            <hardware>
+                <plugin>gazebo_ros2_control/GazeboSystem</plugin>
+            </hardware>
+            <joint name="joint_5">
+                <param name="mimic">joint_4</param>
+                <param name="multiplier">-1</param>
+                <command_interface name="position">
+                    <param name="min">0.0</param>
+                    <param name="max">${PI/2}</param>
+                </command_interface>
+            </joint>
+        </xacro:if>
+        <xacro:unless value="$(arg is_sim)">
+            <hardware>
+                <plugin>arduinobot_controller/ArduinobotInterface</plugin>
+                <param name="port">/dev/ttyUSB0</param>
+            </hardware>
+        </xacro:unless>
         <joint name="joint_1">
             <command_interface name="position">
@@ -34,12 +50,4 @@
             <state_interface name="position"/>
         </joint>
-        <joint name="joint_5">
-            <param name="mimic">joint_4</param>
-            <param name="multiplier">-1</param>
-            <command_interface name="position">
-                <param name="min">0.0</param>
-                <param name="max">${PI/2}</param>
-            </command_interface>
-        </joint>
     </ros2_control>
 </robot>

File: arduinobot_ws/src/install/arduinobot_description/share/arduinobot_description/urdf/arduinobot.urdf.xacro (robot description, xacro)
@@ -219,11 +219,12 @@
         <limit lower="-${PI/2}" upper="0.0" effort="${effort}" velocity="${velocity}"/>
     </joint>
-    <joint name="joint_5" type="revolute" >
+    <joint name ="joint_5" type="revolute">
         <parent link="claw_support"/>
-        <child link="gripper_left"/>
+        <child link = "gripper_left"/>
+        <origin xyz="-0.22 0.13 -0.1"/>
         <axis xyz="0 0 1"/>
-        <origin rpy="0 0 0" xyz="-0.22 0.13 -0.1"/>
+        <limit lower="0.0" upper="${PI / 2}"
+               effort="${effort}" velocity="${velocity}"/>
         <mimic joint="joint_4" multiplier="-1"/>
-        <limit lower="0.0" upper="${PI/2}" effort="${effort}" velocity="${velocity}"/>
     </joint>
     <xacro:default_transmission number="1"/>

File: arduinobot_ws/src/install/arduinobot_description/share/arduinobot_description/urdf/arduinobot_ros2_control.xacro (robot description, xacro)
@@ -41,5 +41,4 @@
                 <param name="max">${PI/2}</param>
             </command_interface>
-            <state_interface name="position"/>
         </joint>
     </ros2_control>
